Commit message: temp

File: src/gazebo_env/model/humanoid.urdf (robot description, URDF)
Before this commit: robot human, 19 links, 18 joints
Links:
- removed link left_arm
- removed link left_hand
- removed link right_arm
- removed link right_hand
Joints:
- removed joint left_arm_lower
- removed joint left_arm_upper
- removed joint right_arm_lower
- removed joint right_arm_upper

File: src/gazebo_env/model/new_left.urdf (robot description, URDF)
Before this commit: robot left_arm, 4 links, 3 joints
Links:
- link chest: mass 0.531912778600973 -> 0.53191; geometry collision mesh filename=meshes/chest.STL; visual mesh filename=meshes/chest.STL
- link left_arm: geometry collision mesh filename=meshes/left_arm.STL; visual mesh filename=meshes/left_arm.STL
- link left_hand: geometry collision mesh filename=meshes/left_hand.STL; visual mesh filename=meshes/left_hand.STL
- link left_shoulder: geometry collision mesh filename=meshes/left_shoulder.STL; visual mesh filename=meshes/left_shoulder.STL
Joints:
- joint left_arm_lower: axis 0 0 0 -> 0 1 0; limit (none) -> lower=0 upper=0 effort=0 velocity=0; origin xyz=0.0247500000000004 -0.11005 0.122 rpy=1.5707963267949 1.5707963267949 0 -> xyz=-0.0281 0.02335 -0.1076 rpy=0 0 0; type fixed -> revolute
- joint left_arm_middle: axis 0 0 0 -> -1 0 0; limit (none) -> lower=0 upper=0 effort=0 velocity=0; origin xyz=0 -0.0241430970576075 0.0348343038500071 rpy=-1.57079632679489 -0.610725964389222 1.5707963267949 -> xyz=0.0281 0.0258 -0.029 rpy=0 0 0; type fixed -> revolute
- joint left_arm_upper: axis 0 0 0 -> 0 1 0; limit (none) -> lower=0 upper=0 effort=0 velocity=0; origin xyz=-0.103502634219692 0.00416746931816645 0.0134 rpy=2.18152229118412 1.5707963267949 0 -> xyz=0.0134 0.0779 0 rpy=0 0 0; type fixed -> revolute
